File: ESC_Motor1.kicad_sch (KiCad schematic)
At the start: 33 parts, among them Q10 FDMS8350LET40, Q11 FDMS8350LET40, Q12 FDMS8350LET40, Q13 FDMS8350LET40, Q15 FDMS8350LET40, Q3 FDMS8350LET40, Q4 FDMS8350LET40, Q5 FDMS8350LET40, Q6 FDMS8350LET40, Q7 FDMS8350LET40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

Commit message: motor esc schematics
Parts:
- removed Q12, Q13, Q3, Q5, Q8, Q9: FDMS8350LET40, Package_TO_SOT_SMD:TDSON-8-1, symbol Transistor_FET:FDMS8350LET40
- removed R30, R31, R36, R37, R40, R41: 10, Resistor_SMD:R_0805_2012Metric_Pad1.20x1.40mm_HandSolder, symbol Device:R_Small_US
Connections:
- net ESC_M1_PHASE_1_LOW: no longer Q11.1 (S), Q11.2 (S), Q11.3 (S), Q4.1 (S), Q4.2 (S), Q4.3 (S), Q7.1 (S), Q7.2 (S), Q7.3 (S)
- net ESC_M1_PHASE_3_HIGH: now also R38.1; no longer R39.1
- net ESC_M1_PHASE_3_LOW: now also R39.1; no longer R38.1
- net ESC_VBAT+: now reaches Q6.5 (D)
- net ESC_VBAT+: now also Q10.5 (D), Q15.5 (D)
- new net ESC_HBRIDGE_OUT: Q11.1 (S), Q11.2 (S), Q11.3 (S), Q4.1 (S), Q4.2 (S), Q4.3 (S), Q7.1 (S), Q7.2 (S), Q7.3 (S)
Other:
- note removed: "S"
