File: ESC_Motor2.kicad_sch (KiCad schematic)
At the start: 33 parts, among them Q14 FDMS8350LET40, Q16 FDMS8350LET40, Q17 FDMS8350LET40, Q18 FDMS8350LET40, Q19 FDMS8350LET40, Q20 FDMS8350LET40, Q21 FDMS8350LET40, Q22 FDMS8350LET40, Q23 FDMS8350LET40, Q24 FDMS8350LET40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

Commit message: motor esc schematics
Parts:
- removed Q21, Q22, Q23, Q24, Q25, Q26: FDMS8350LET40, Package_TO_SOT_SMD:TDSON-8-1, symbol Transistor_FET:FDMS8350LET40
- removed R53, R54, R55, R56, R57, R58: 10, Resistor_SMD:R_0805_2012Metric_Pad1.20x1.40mm_HandSolder, symbol Device:R_Small_US
Connections:
- net ESC_M2_PHASE_1_LOW: no longer Q16.1 (S), Q16.2 (S), Q16.3 (S), Q18.1 (S), Q18.2 (S), Q18.3 (S), Q20.1 (S), Q20.2 (S), Q20.3 (S)
- net ESC_M2_PHASE_3_HIGH: now also R51.1; no longer R52.1
- net ESC_M2_PHASE_3_LOW: now also R52.1; no longer R51.1
- net ESC_VBAT+: now reaches Q14.5 (D)
- net ESC_VBAT+: now also Q17.5 (D), Q19.5 (D)
- new net ESC_HBRIDGE_OUT: Q16.1 (S), Q16.2 (S), Q16.3 (S), Q18.1 (S), Q18.2 (S), Q18.3 (S), Q20.1 (S), Q20.2 (S), Q20.3 (S)
Other:
- note removed: "S"
