File: ESC_Motor3.kicad_sch (KiCad schematic)
At the start: 33 parts, among them Q27 FDMS8350LET40, Q28 FDMS8350LET40, Q29 FDMS8350LET40, Q30 FDMS8350LET40, Q31 FDMS8350LET40, Q32 FDMS8350LET40, Q33 FDMS8350LET40, Q34 FDMS8350LET40, Q35 FDMS8350LET40, Q36 FDMS8350LET40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

Commit message: motor esc schematics
Parts:
- removed Q33, Q34, Q35, Q36, Q37, Q38: FDMS8350LET40, Package_TO_SOT_SMD:TDSON-8-1, symbol Transistor_FET:FDMS8350LET40
- removed R66, R67, R68, R69, R70, R71: 10, Resistor_SMD:R_0805_2012Metric_Pad1.20x1.40mm_HandSolder, symbol Device:R_Small_US
Connections:
- net ESC_M3_PHASE_1_LOW: no longer Q28.1 (S), Q28.2 (S), Q28.3 (S), Q30.1 (S), Q30.2 (S), Q30.3 (S), Q32.1 (S), Q32.2 (S), Q32.3 (S)
- net ESC_M3_PHASE_3_HIGH: now also R64.1; no longer R65.1
- net ESC_M3_PHASE_3_LOW: now also R65.1; no longer R64.1
- net ESC_VBAT+: now reaches Q27.5 (D)
- net ESC_VBAT+: now also Q29.5 (D), Q31.5 (D)
- new net ESC_HBRIDGE_OUT: Q28.1 (S), Q28.2 (S), Q28.3 (S), Q30.1 (S), Q30.2 (S), Q30.3 (S), Q32.1 (S), Q32.2 (S), Q32.3 (S)
Other:
- note removed: "S"
