File: ESC_Motor4.kicad_sch (KiCad schematic)
At the start: 0 parts

Commit message: motor esc schematics
Parts:
- added C55: 10uF, Capacitor_SMD:C_0805_2012Metric_Pad1.18x1.45mm_HandSolder, symbol Device:C
- added C56: 100nF, Capacitor_SMD:C_0805_2012Metric_Pad1.18x1.45mm_HandSolder, symbol Device:C
- added C57, C58, C59: 220nF, Capacitor_SMD:C_0805_2012Metric_Pad1.18x1.45mm_HandSolder, symbol Device:C
- added D18, D19, D20: BAS21, Package_TO_SOT_SMD:SOT-23, symbol Diode:BAS21
- added Q39, Q40, Q41, Q42, Q43, Q44: FDMS8350LET40, Package_TO_SOT_SMD:TDSON-8-1, symbol Transistor_FET:FDMS8350LET40
- added R72, R73, R74, R75, R76, R77: 10, Resistor_SMD:R_0805_2012Metric_Pad1.20x1.40mm_HandSolder, symbol Device:R_Small_US
- added U16: FD6288Q, FD6288Q:QFN50P400X400X90-25N, symbol FD6288Q:FD6288Q
Connections:
- new net: Q43.4 (G), R76.2
- new net: Q42.4 (G), R75.2
- new net: Q40.4 (G), R73.2
- new net: Q39.4 (G), R72.2
- new net: Q44.4 (G), R77.2
- new net: Q41.4 (G), R74.2
- new net ESC_COM: C55.2, C56.2, U16.25 (EXP), U16.6 (COM)
- new net ESC_HBRIDGE_OUT: Q40.1 (S), Q40.2 (S), Q40.3 (S), Q42.1 (S), Q42.2 (S), Q42.3 (S), Q44.1 (S), Q44.2 (S), Q44.3 (S), R73.1, U16.11 (LO1)
- new net ESC_M4_HIN1: U16.22 (HIN1)
- new net ESC_M4_HIN2: U16.23 (HIN2)
- new net ESC_M4_HIN3: U16.24 (HIN3)
- new net ESC_M4_LIN1: U16.1 (LIN1)
- new net ESC_M4_LIN2: U16.2 (LIN2)
- new net ESC_M4_LIN3: U16.3 (LIN3)
- new net ESC_M4_PHASE_1: C57.1, Q39.1 (S), Q39.2 (S), Q39.3 (S), Q40.5 (D), U16.18 (VS1)
- new net ESC_M4_PHASE_1_HIGH: R72.1, U16.19 (HO1)
- new net ESC_M4_PHASE_2: C58.1, Q41.1 (S), Q41.2 (S), Q41.3 (S), Q42.5 (D), U16.15 (VS2)
- new net ESC_M4_PHASE_2_HIGH: R74.1, U16.16 (HO2)
- new net ESC_M4_PHASE_2_LOW: R75.1, U16.10 (LO2)
- new net ESC_M4_PHASE_3: C59.1, Q43.1 (S), Q43.2 (S), Q43.3 (S), Q44.5 (D), U16.12 (VS3)
- new net ESC_M4_PHASE_3_HIGH: R76.1, U16.13 (HO3)
- new net ESC_M4_PHASE_3_LOW: R77.1, U16.9 (LO3)
- new net ESC_M4_VB1: C57.2, D18.3 (K), U16.20 (VB1)
- new net ESC_M4_VB2: C58.2, D19.3 (K), U16.17 (VB2)
- new net ESC_M4_VB3: C59.2, D20.3 (K), U16.14 (VB3)
- new net ESC_VBAT+: Q39.5 (D), Q41.5 (D), Q43.5 (D)
- new net ESC_VCC: C55.1, C56.1, D18.1 (A), D19.1 (A), D20.1 (A), U16.4 (VCC)
Other:
- note added: "10-12v"
- note added: "Motor 4"
- note added: "X7R"
