File: esc.kicad_sch (KiCad schematic)
At the start: 17 parts, among them U10 INA181, U2 STM32G071G8U6N, U8 TLV75733PDBV

Commit message: motor esc schematics
Parts:
- removed U2: STM32G071G8U6N, Package_DFN_QFN:QFN-28_4x4mm_P0.5mm, symbol MCU_ST_STM32G0:STM32G071G8UxN
- added C60, C61, C62, C63, C65, C66: 100nF, Capacitor_SMD:C_0805_2012Metric_Pad1.18x1.45mm_HandSolder, symbol Device:C
- added C64: 1uF, Capacitor_SMD:C_0805_2012Metric_Pad1.18x1.45mm_HandSolder, symbol Device:C
- added D21: 3.3V LED, LED_SMD:LED_0402_1005Metric, symbol Device:LED
- added J10: Debug, Connector_PinHeader_2.54mm:PinHeader_1x05_P2.54mm_Vertical, symbol Connector:Conn_01x05_Pin
- added J16: To FC, symbol Connector:Conn_01x07_Pin
- added J17: From BEC, Connector_Hirose:Hirose_DF13-02P-1.25DS_1x02_P1.25mm_Horizontal, symbol Connector:Conn_01x02_Pin
- added R59: 10k, Resistor_SMD:R_0603_1608Metric_Pad0.98x0.95mm_HandSolder, symbol Device:R_Small_US
- added R84: 10K, Resistor_SMD:R_0603_1608Metric_Pad0.98x0.95mm_HandSolder, symbol Device:R
- added U17: STM32F303C8T6, Package_QFP:LQFP-48_7x7mm_P0.5mm, symbol MCU_ST_STM32F3:STM32F303C8Tx
- added Y3: 8 MHz, Crystal:Resonator_SMD_Murata_CSTxExxV-3Pin_3.0x1.1mm, symbol Device:Resonator
- R29: value 1m -> 0.5m
- R44: value 100k -> 50k
Connections:
- net ESC_3.3V: now also C60.1, C61.1, C62.1, C63.1, C64.1, C65.2, J10.5 (Pin_5), U17.1 (VBAT), U17.24 (VDD), U17.36 (VDD), U17.48 (VDD), U17.9 (VDDA)
- net ESC_5V: now also J17.1 (Pin_1)
- net ESC_COM: now also C60.2, C61.2, C62.2, C63.2, C64.2, C65.1, D21.1 (K), J10.4 (Pin_4), J16.1 (Pin_1), J17.2 (Pin_2), R59.2, U17.23 (VSS), U17.35 (VSS), U17.47 (VSS), U17.8 (VSSA), Y3.2
- net ESC_CURRENTSENSE: now also U17.10 (PA0)
- net ESC_UNSAFE_VBAT+: now reaches D8.1 (A1)
- net ESC_UNSAFE_VBAT+: now also R44.1
- net ESC_UNSAFE_VBAT-: now reaches D8.2 (A2)
- net ESC_UNSAFE_VBAT-: now also R45.2
- net ESC_NRST: now reaches C42.1, R46.2
- net ESC_NRST: now also J10.3 (Pin_3), U17.7 (NRST)
- net ESC_VBATSENSE: now reaches R44.2, R45.1
- net ESC_VBATSENSE: now also U17.11 (PA1)
- net at R29.2, U10.3 (+): now also C66.1
- net at R29.3, U10.4 (-): now also C66.2
- net HBRIDGE_OUT renamed ESC_HBRIDGE_OUT
- new net: D21.2 (A), R84.2
- new net: R84.1, U17.4 (PC15)
- new net: U17.5 (PF0), Y3.1
- new net: U17.6 (PF1), Y3.3
- new net DSHOT1: J16.2 (Pin_2), U17.32 (PA11)
- new net DSHOT2: J16.3 (Pin_3), U17.33 (PA12)
- new net DSHOT3: J16.4 (Pin_4), U17.2 (PC13)
- new net DSHOT4: J16.5 (Pin_5), U17.3 (PC14)
- new net ESC_BOOT0: R59.1, U17.44 (BOOT0)
- new net ESC_M1_HIN1: U17.12 (PA2)
- new net ESC_M1_HIN2: U17.14 (PA4)
- new net ESC_M1_HIN3: U17.16 (PA6)
- new net ESC_M1_LIN1: U17.13 (PA3)
- new net ESC_M1_LIN2: U17.15 (PA5)
- new net ESC_M1_LIN3: U17.17 (PA7)
- new net ESC_M2_HIN1: U17.29 (PA8)
- new net ESC_M2_HIN2: U17.31 (PA10)
- new net ESC_M2_HIN3: U17.19 (PB1)
- new net ESC_M2_LIN1: U17.30 (PA9)
- new net ESC_M2_LIN2: U17.18 (PB0)
- new net ESC_M2_LIN3: U17.20 (PB2)
- new net ESC_M3_HIN1: U17.40 (PB4)
- new net ESC_M3_HIN2: U17.42 (PB6)
- new net ESC_M3_HIN3: U17.45 (PB8)
- new net ESC_M3_LIN1: U17.41 (PB5)
- new net ESC_M3_LIN2: U17.43 (PB7)
- new net ESC_M3_LIN3: U17.46 (PB9)
- new net ESC_M4_HIN1: U17.21 (PB10)
- new net ESC_M4_HIN2: U17.25 (PB12)
- new net ESC_M4_HIN3: U17.27 (PB14)
- new net ESC_M4_LIN1: U17.22 (PB11)
- new net ESC_M4_LIN2: U17.26 (PB13)
- new net ESC_M4_LIN3: U17.28 (PB15)
- new net ESC_SYS_JTCK-SWCLK: J10.2 (Pin_2), U17.37 (PA14)
- new net ESC_SYS_JTMS-SWDIO: J10.1 (Pin_1), U17.34 (PA13)
- new net ESC_UART_RX: J16.7 (Pin_7), U17.38 (PA15)
- new net ESC_UART_TX: J16.6 (Pin_6), U17.39 (PB3)
Other:
- added sheet ESC_Motor3 (ESC_Motor3.kicad_sch)
- added sheet ESC_Motor4 (ESC_Motor4.kicad_sch)
- note added: "0.0005 Ω"
- note added: "2512 package"
- note added: "3W rated"
- note added: "A1"
- note added: "Current-Sense Type"
- note removed: "A2"
- note removed: "Not 1M"
- moved on the sheet: C40, C41, C42, C43, C44, D11, D8, R29, R42, R43, R44, R45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
