File: customDevboard.kicad_pcb (KiCad board)
At the start: 4 copper layers, 40 x 40 mm, 111 parts, among them J1 From BEC, J10 PA4, J11 PB2, J12 PC11, J13 PC10, J14 PB6, J15 PB7, J16 PA9, J17 PA10, J18 PA2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

Commit message: add Dreamscape F722 Silkscreen
Other:
- board text added: "DREAMSCAPE F722 V1.0"
- board text added: "DS-F722-V1.0"
- board text removed: "FC P1"
