File: customDevboard.kicad_sch (KiCad schematic)
At the start: 92 parts, among them J1 From BEC, J10 PA4, J11 PB2, J12 PC11, J13 PC10, J14 PB6, J15 PB7, J16 PA9, J17 PA10, J18 PA2, J19 PA3, J2 BZ+, J20 PB10, J21 PB11, J22 USB_C_Receptacle_USB2.0_14P, J23 To GPS, J24 Debug, J25 Conn_01x01, J26 Conn_01x01, J27 Conn_01x01, J28 PA0, J29 PA1, J3 COL, J30 Conn_01x01, J31 Conn_01x01, J32 Conn_01x01, J33 Conn_01x01, J34 Conn_01x01, J35 Conn_01x01, J36 Conn_01x01, J37 Conn_01x01, J38 Conn_01x01, J39 Conn_01x01, J4 PA7, J40 Conn_01x01, J41 Conn_01x01, J42 Conn_01x01, J43 Conn_01x01, J44 Conn_01x01, J5 PA6, J6 PA5, J7 PC1, J8 PC11, J9 PB13, Q1 AO3401A, Q2 BC817, SW1 CK_KMS2xxGP, SW2 CK_KMS2xxGP, U1 STM32F722RET6, U2 TLV75733PDRV, U3 TPD2EUSB30, Y1 8MHz, Y2 32.768KHz

Commit message: ready for ship
Parts:
- removed J23: To GPS, Connector_Hirose:Hirose_DF13-06P-1.25DS_1x06_P1.25mm_Horizontal, symbol Connector:Conn_01x06_Pin
- removed J24: Debug, Connector_PinHeader_2.54mm:PinHeader_1x03_P2.54mm_Vertical, symbol Connector:Conn_01x03_Pin
- removed SW1, SW2: CK_KMS2xxGP, Button_Switch_SMD:SW_SPST_CK_KMS2xxGP, symbol Switch:CK_KMS2xxGP
- added J23: SWDIO, Connector_Wire:SolderWirePad_1x01_SMD_1x2mm, symbol Connector_Generic:Conn_01x01
- added J24: SWCLK, Connector_Wire:SolderWirePad_1x01_SMD_1x2mm, symbol Connector_Generic:Conn_01x01
- added SW1, SW2: SW_SPST, Button_Switch_SMD:SW_SPST_B3U-3000P, symbol Switch:SW_SPST
Connections:
- net +3.3V: now also SW2.2 (B)
- net BOOT0: now also SW2.1 (A)
- net GND: now also SW1.2 (B)
- net NRST: now also SW1.1 (A)
- net SYS_JTCK-SWCLK: now also J24.1 (Pin_1)
- net SYS_JTMS-SWDIO: now also J23.1 (Pin_1)
Other:
- note removed: "GND"
- note removed: "SWCLK"
- note removed: "SWDIO"

Commit message: add Dreamscape F722 Silkscreen
Other:
- note added: "Dreamscape F722"
Changed lines of the file:
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@@
+		)
+	)
+	(text "Dreamscape F722"
+		(exclude_from_sim no)
+		(at 195.326 189.738 0)
+		(effects
+			(font
+				(size 1.27 1.27)
+			)
 		)
 	)
