File: kicad/Dreamscape-F722.kicad_sch (KiCad schematic)
At the start: 92 parts, among them J1 From BEC, J10 PA4, J11 PB2, J12 PC11, J13 PC10, J14 PB6, J15 PB7, J16 PA9, J17 PA10, J18 PA2, J19 PA3, J2 BZ+, J20 PB10, J21 PB11, J22 USB_C_Receptacle_USB2.0_14P, J23 SWDIO, J24 SWCLK, J25 Conn_01x01, J26 Conn_01x01, J27 Conn_01x01, J28 PA0, J29 PA1, J3 COL, J30 Conn_01x01, J31 Conn_01x01, J32 Conn_01x01, J33 Conn_01x01, J34 Conn_01x01, J35 Conn_01x01, J36 Conn_01x01, J37 Conn_01x01, J38 Conn_01x01, J39 Conn_01x01, J4 PA7, J40 Conn_01x01, J41 Conn_01x01, J42 Conn_01x01, J43 Conn_01x01, J44 Conn_01x01, J5 PA6, J6 PA5, J7 PC1, J8 PC11, J9 PB13, Q1 AO3401A, Q2 BC817, SW1 SW_SPST, SW2 SW_SPST, U1 STM32F722RET6, U2 TLV75733PDRV, U3 TPD2EUSB30, Y1 8MHz, Y2 32.768KHz

Commit message: move imported parts into kicad directory
Parts:
- added D3, D4: SS14, Diode_SMD:D_SMA, symbol Diode:SS14
Connections:
- net +5V: now also D3.1 (K), D4.1 (K); no longer J2.1 (Pin_1)
- net VBUS: no longer names the net of J22.A4 (VBUS), J22.A9 (VBUS), J22.B4 (VBUS), J22.B9 (VBUS)
- net VBUS: now also D4.2 (A)
- new net: D3.2 (A), J2.1 (Pin_1)
Changed lines of the file:
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@@
 	(wire
 		(pts
+			(xy 251.46 114.3) (xy 251.46 115.57)
+		)
+		(stroke
+			(width 0)
+			(type default)
+		)
+	)
+	(wire
+		(pts
 			(xy 106.68 69.85) (xy 106.68 68.58)
 		)
@@
 	(wire
 		(pts
-			(xy 93.98 25.4) (xy 92.71 25.4)
+			(xy 104.14 25.4) (xy 101.6 25.4)
 		)
 		(stroke
@@
 	(wire
 		(pts
-			(xy 241.3 113.03) (xy 241.3 115.57)
-		)
-		(stroke
-			(width 0)
-			(type default)
-		)
-	)
-	(wire
-		(pts
 			(xy 48.26 143.51) (xy 63.5 143.51)
 		)
@@
 	(wire
 		(pts
+			(xy 93.98 25.4) (xy 92.71 25.4)
+		)
+		(stroke
+			(width 0)
+			(type default)
+		)
+	)
+	(wire
+		(pts
 			(xy 149.86 105.41) (xy 151.13 105.41)
 		)
@@
 	(wire
 		(pts
+			(xy 248.92 115.57) (xy 251.46 115.57)
+		)
+		(stroke
+			(width 0)
+			(type default)
+		)
+	)
+	(wire
+		(pts
 			(xy 104.14 128.27) (xy 105.41 128.27)
 		)
@@
 	(wire
 		(pts
-			(xy 93.98 24.13) (xy 93.98 25.4)
+			(xy 104.14 25.4) (xy 104.14 24.13)
 		)
 		(stroke
@@
 	)
 	(symbol
-		(lib_id "power:VBUS")
-		(at 241.3 113.03 0)
-		(unit 1)
-		(exclude_from_sim no)
-		(in_bom yes)
-		(on_board yes)
-		(dnp no)
-		(fields_autoplaced yes)
-		(property "Reference" "#PWR030"
-			(at 241.3 116.84 0)
-			(effects
-				(font
-					(size 1.27 1.27)
-				)
-				(hide yes)
-			)
-		)
-		(property "Value" "VBUS"
-			(at 241.3 107.95 0)
-			(effects
-				(font
-					(size 1.27 1.27)
-				)
-			)
-		)
-		(property "Footprint" ""
-			(at 241.3 113.03 0)
-			(effects
-				(font
-					(size 1.27 1.27)
-				)
-				(hide yes)
-			)
-		)
-		(property "Datasheet" ""
-			(at 241.3 113.03 0)
-			(effects
-				(font
-					(size 1.27 1.27)
-				)
-				(hide yes)
-			)
-		)
-		(property "Description" "Power symbol creates a global label with name \"VBUS\""
-			(at 241.3 113.03 0)
-			(effects
-				(font
-					(size 1.27 1.27)
-				)
-				(hide yes)
-			)
-		)
-		(pin "1"
-		)
-		(instances
-			(project ""
-				(path "/87078d80-bd64-4f8e-8d0b-a79df4010aa3"
-					(reference "#PWR030")
-					(unit 1)
-				)
-			)
-		)
-	)
-	(symbol
 		(lib_id "Device:R_Small_US")
 		(at 242.57 120.65 90)
@@
 	)
 	(symbol
+		(lib_id "Diode:SS14")
+		(at 245.11 115.57 180)
+		(unit 1)
+		(exclude_from_sim no)
+		(in_bom yes)
+		(on_board yes)
+		(dnp no)
+		(fields_autoplaced yes)
+		(property "Reference" "D4"
+			(at 245.4275 109.22 0)
+			(effects
+				(font
+					(size 1.27 1.27)
+				)
+			)
+		)
+		(property "Value" "SS14"
+			(at 245.4275 111.76 0)
+			(effects
+				(font
+					(size 1.27 1.27)
+				)
+			)
+		)
+		(property "Footprint" "Diode_SMD:D_SMA"
+			(at 245.11 111.125 0)
+			(effects
+				(font
+					(size 1.27 1.27)
+				)
+				(hide yes)
+			)
+		)
+		(property "Datasheet" "https://www.vishay.com/docs/88746/ss12.pdf"
+			(at 245.11 115.57 0)
+			(effects
+				(font
+					(size 1.27 1.27)
+				)
+				(hide yes)
+			)
+		)
+		(property "Description" "40V 1A Schottky Diode, SMA"
+			(at 245.11 115.57 0)
+			(effects
+				(font
+					(size 1.27 1.27)
+				)
+				(hide yes)
+			)
+		)
+		(pin "2"
+		)
+		(pin "1"
+		)
+		(instances
+			(project "Dreamscape-F722"
+				(path "/87078d80-bd64-4f8e-8d0b-a79df4010aa3"
+					(reference "D4")
+					(unit 1)
+				)
+			)
+		)
+	)
+	(symbol
 		(lib_id "Device:C")
 		(at 20.32 130.81 0)
@@
 	)
 	(symbol
+		(lib_id "Diode:SS14")
+		(at 97.79 25.4 180)
+		(unit 1)
+		(exclude_from_sim no)
+		(in_bom yes)
+		(on_board yes)
+		(dnp no)
+		(fields_autoplaced yes)
+		(property "Reference" "D3"
+			(at 98.1075 19.05 0)
+			(effects
+				(font
+					(size 1.27 1.27)
+				)
+			)
+		)
+		(property "Value" "SS14"
+			(at 98.1075 21.59 0)
+			(effects
+				(font
+					(size 1.27 1.27)
+				)
+			)
+		)
+		(property "Footprint" "Diode_SMD:D_SMA"
+			(at 97.79 20.955 0)
+			(effects
+				(font
+					(size 1.27 1.27)
+				)
+				(hide yes)
+			)
+		)
+		(property "Datasheet" "https://www.vishay.com/docs/88746/ss12.pdf"
+			(at 97.79 25.4 0)
+			(effects
+				(font
+					(size 1.27 1.27)
+				)
+				(hide yes)
+			)
+		)
+		(property "Description" "40V 1A Schottky Diode, SMA"
+			(at 97.79 25.4 0)
+			(effects
+				(font
+					(size 1.27 1.27)
+				)
+				(hide yes)
+			)
+		)
+		(pin "2"
+		)
+		(pin "1"
+		)
+		(instances
+			(project ""
+				(path "/87078d80-bd64-4f8e-8d0b-a79df4010aa3"
+					(reference "D3")
+					(unit 1)
+				)
+			)
+		)
+	)
+	(symbol
 		(lib_id "MCU_ST_STM32F7:STM32F722RETx")
 		(at 83.82 133.35 0)
@@
 	(symbol
 		(lib_id "power:+5V")
-		(at 93.98 24.13 0)
+		(at 104.14 24.13 0)
 		(unit 1)
 		(exclude_from_sim no)
@@
 		(fields_autoplaced yes)
 		(property "Reference" "#PWR013"
-			(at 93.98 27.94 0)
+			(at 104.14 27.94 0)
 			(effects
 				(font
@@
 		)
 		(property "Value" "+5V"
-			(at 93.98 19.05 0)
+			(at 104.14 19.05 0)
 			(effects
 				(font
@@
 		)
 		(property "Footprint" ""
-			(at 93.98 24.13 0)
+			(at 104.14 24.13 0)
 			(effects
 				(font
@@
 		)
 		(property "Datasheet" ""
-			(at 93.98 24.13 0)
+			(at 104.14 24.13 0)
 			(effects
 				(font
@@
 		)
 		(property "Description" "Power symbol creates a global label with name \"+5V\""
-			(at 93.98 24.13 0)
+			(at 104.14 24.13 0)
 			(effects
 				(font
@@
 					(unit 1)
 				)
+			)
+		)
+	)
+	(symbol
+		(lib_id "power:+5V")
+		(at 251.46 114.3 0)
+		(unit 1)
+		(exclude_from_sim no)
+		(in_bom yes)
+		(on_board yes)
+		(dnp no)
+		(fields_autoplaced yes)
+		(property "Reference" "#PWR020"
+			(at 251.46 118.11 0)
+			(effects
+				(font
+					(size 1.27 1.27)
+				)
+				(hide yes)
+			)
+		)
+		(property "Value" "+5V"
+			(at 251.46 109.22 0)
+			(effects
+				(font
+					(size 1.27 1.27)
+				)
+			)
+		)
+		(property "Footprint" ""
+			(at 251.46 114.3 0)
+			(effects
+				(font
+					(size 1.27 1.27)
+				)
+				(hide yes)
+			)
+		)
+		(property "Datasheet" ""
+			(at 251.46 114.3 0)
+			(effects
+				(font
+					(size 1.27 1.27)
+				)
+				(hide yes)
+			)
+		)
+		(property "Description" "Power symbol creates a global label with name \"+5V\""
+			(at 251.46 114.3 0)
+			(effects
+				(font
+					(size 1.27 1.27)
+				)
+				(hide yes)
+			)
+		)
+		(pin "1"
+		)
+		(instances
+			(project ""
+				(path "/87078d80-bd64-4f8e-8d0b-a79df4010aa3"
+					(reference "#PWR020")
+					(unit 1)
+				)

Commit message: update repos
Connections:
- net +5V: now also J2.1 (Pin_1); no longer Q1.3 (D)
- net at D3.2 (A): now also Q1.3 (D); no longer J2.1 (Pin_1)
Other:
- moved on the sheet: D3, J1, Q1, R3
Changed lines of the file:
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@@
 	(text "PMOS Reverse\nPolarity Protection"
 		(exclude_from_sim no)
-		(at 59.182 23.622 0)
+		(at 60.452 28.448 0)
 		(effects
 			(font
@@
 	)
 	(junction
-		(at 40.64 35.56)
+		(at 44.45 36.83)
 		(diameter 0)
 		(color 0 0 0 0)
@@
 	(wire
 		(pts
-			(xy 40.64 27.94) (xy 40.64 29.21)
+			(xy 44.45 29.21) (xy 44.45 30.48)
 		)
 		(stroke
@@
 	(wire
 		(pts
-			(xy 104.14 25.4) (xy 101.6 25.4)
-		)
-		(stroke
-			(width 0)
-			(type default)
-		)
-	)
-	(wire
-		(pts
 			(xy 90.17 36.83) (xy 90.17 38.1)
 		)
@@
 	(wire
 		(pts
-			(xy 40.64 35.56) (xy 40.64 34.29)
+			(xy 44.45 36.83) (xy 44.45 35.56)
 		)
 		(stroke
@@
 	(wire
 		(pts
-			(xy 34.29 20.32) (xy 35.56 20.32)
+			(xy 38.1 21.59) (xy 39.37 21.59)
 		)
 		(stroke
@@
 	(wire
 		(pts
-			(xy 40.64 35.56) (xy 49.53 35.56)
-		)
-		(stroke
-			(width 0)
-			(type default)
-		)
-	)
-	(wire
-		(pts
 			(xy 123.19 77.47) (xy 123.19 78.74)
 		)
@@
 	(wire
 		(pts
+			(xy 44.45 38.1) (xy 44.45 36.83)
+		)
+		(stroke
+			(width 0)
+			(type default)
+		)
+	)
+	(wire
+		(pts
 			(xy 104.14 173.99) (xy 127 173.99)
 		)
@@
 	(wire
 		(pts
+			(xy 92.71 25.4) (xy 99.06 25.4)
+		)
+		(stroke
+			(width 0)
+			(type default)
+		)
+	)
+	(wire
+		(pts
 			(xy 104.14 97.79) (xy 105.41 97.79)
 		)
@@
 	(wire
 		(pts
-			(xy 34.29 25.4) (xy 34.29 20.32)
+			(xy 38.1 26.67) (xy 38.1 21.59)
 		)
 		(stroke
@@
 	(wire
 		(pts
-			(xy 26.67 25.4) (xy 34.29 25.4)
+			(xy 30.48 26.67) (xy 38.1 26.67)
 		)
 		(stroke
@@
 	(wire
 		(pts
-			(xy 26.67 27.94) (xy 34.29 27.94)
+			(xy 30.48 29.21) (xy 38.1 29.21)
 		)
 		(stroke
@@
 	(wire
 		(pts
-			(xy 45.72 20.32) (xy 49.53 20.32)
+			(xy 49.53 21.59) (xy 50.8 21.59)
 		)
 		(stroke
@@
 	(wire
 		(pts
-			(xy 93.98 25.4) (xy 92.71 25.4)
-		)
-		(stroke
-			(width 0)
-			(type default)
-		)
-	)
-	(wire
-		(pts
 			(xy 149.86 105.41) (xy 151.13 105.41)
 		)
@@
 	(wire
 		(pts
-			(xy 34.29 27.94) (xy 34.29 35.56)
+			(xy 38.1 29.21) (xy 38.1 36.83)
 		)
 		(stroke
@@
 	(wire
 		(pts
+			(xy 60.96 21.59) (xy 58.42 21.59)
+		)
+		(stroke
+			(width 0)
+			(type default)
+		)
+	)
+	(wire
+		(pts
 			(xy 104.14 143.51) (xy 127 143.51)
 		)
@@
 	(wire
 		(pts
-			(xy 34.29 35.56) (xy 40.64 35.56)
+			(xy 38.1 36.83) (xy 44.45 36.83)
 		)
 		(stroke
@@
 	(wire
 		(pts
-			(xy 104.14 25.4) (xy 104.14 24.13)
+			(xy 99.06 25.4) (xy 99.06 24.13)
 		)
 		(stroke
@@
 	(symbol
 		(lib_id "power:GND")
-		(at 49.53 35.56 0)
+		(at 44.45 38.1 0)
 		(unit 1)
 		(exclude_from_sim no)
@@
 		(fields_autoplaced yes)
 		(property "Reference" "#PWR09"
-			(at 49.53 41.91 0)
+			(at 44.45 44.45 0)
 			(effects
 				(font
@@
 		)
 		(property "Value" "GND"
-			(at 49.53 40.64 0)
+			(at 44.45 43.18 0)
 			(effects
 				(font
@@
 		)
 		(property "Footprint" ""
-			(at 49.53 35.56 0)
+			(at 44.45 38.1 0)
 			(effects
 				(font
@@
 		)
 		(property "Datasheet" ""
-			(at 49.53 35.56 0)
+			(at 44.45 38.1 0)
 			(effects
 				(font
@@
 		)
 		(property "Description" "Power symbol creates a global label with name \"GND\" , ground"
-			(at 49.53 35.56 0)
+			(at 44.45 38.1 0)
 			(effects
 				(font
@@
 	(symbol
 		(lib_id "Connector:Conn_01x02_Pin")
-		(at 21.59 25.4 0)
+		(at 25.4 26.67 0)
 		(unit 1)
 		(exclude_from_sim no)
@@
 		(dnp no)
 		(property "Reference" "J1"
-			(at 20.32 25.3999 0)
+			(at 24.13 26.6699 0)
 			(effects
 				(font
@@
 		)
 		(property "Value" "From BEC"
-			(at 20.32 27.9399 0)
+			(at 24.13 29.2099 0)
 			(effects
 				(font
@@
 		)
 		(property "Footprint" "Connector_Hirose:Hirose_DF13-02P-1.25DS_1x02_P1.25mm_Horizontal"
-			(at 21.59 25.4 0)
+			(at 25.4 26.67 0)
 			(effects
 				(font
@@
 		)
 		(property "Datasheet" "~"
-			(at 21.59 25.4 0)
+			(at 25.4 26.67 0)
 			(effects
 				(font
@@
 		)
 		(property "Description" "Generic connector, single row, 01x02, script generated"
-			(at 21.59 25.4 0)
+			(at 25.4 26.67 0)
 			(effects
 				(font
@@
 	(symbol
 		(lib_id "Transistor_FET:AO3401A")
-		(at 40.64 22.86 270)
+		(at 44.45 24.13 270)
 		(mirror x)
 		(unit 1)
@@
 		(dnp no)
 		(property "Reference" "Q1"
-			(at 40.64 13.97 90)
+			(at 44.45 15.24 90)
 			(effects
 				(font
@@
 		)
 		(property "Value" "AO3401A"
-			(at 40.64 16.51 90)
+			(at 44.45 17.78 90)
 			(effects
 				(font
@@
 		)
 		(property "Footprint" "Package_TO_SOT_SMD:SOT-23"
-			(at 38.735 17.78 0)
+			(at 42.545 19.05 0)
 			(effects
 				(font
@@
 		)
 		(property "Datasheet" "http://www.aosmd.com/pdfs/datasheet/AO3401A.pdf"
-			(at 36.83 17.78 0)
+			(at 40.64 19.05 0)
 			(effects
 				(font
@@
 		)
 		(property "Description" "-4.0A Id, -30V Vds, P-Channel MOSFET, SOT-23"
-			(at 40.64 22.86 0)
+			(at 44.45 24.13 0)
 			(effects
 				(font
@@
 	(symbol
 		(lib_id "power:+5V")
-		(at 49.53 20.32 0)
+		(at 60.96 21.59 0)
 		(unit 1)
 		(exclude_from_sim no)
@@
 		(fields_autoplaced yes)
 		(property "Reference" "#PWR08"
-			(at 49.53 24.13 0)
+			(at 60.96 25.4 0)
 			(effects
 				(font
@@
 		)
 		(property "Value" "+5V"
-			(at 49.53 15.24 0)
+			(at 60.96 16.51 0)
 			(effects
 				(font
@@
 		)
 		(property "Footprint" ""
-			(at 49.53 20.32 0)
+			(at 60.96 21.59 0)
 			(effects
 				(font
@@
 		)
 		(property "Datasheet" ""
-			(at 49.53 20.32 0)
+			(at 60.96 21.59 0)
 			(effects
 				(font
@@
 		)
 		(property "Description" "Power symbol creates a global label with name \"+5V\""
-			(at 49.53 20.32 0)
+			(at 60.96 21.59 0)
 			(effects
 				(font
@@
 	(symbol
 		(lib_id "Diode:SS14")
-		(at 97.79 25.4 180)
+		(at 54.61 21.59 180)
 		(unit 1)
 		(exclude_from_sim no)
@@
 		(fields_autoplaced yes)
 		(property "Reference" "D3"
-			(at 98.1075 19.05 0)
+			(at 54.9275 15.24 0)
 			(effects
 				(font
@@
 		)
 		(property "Value" "SS14"
-			(at 98.1075 21.59 0)
+			(at 54.9275 17.78 0)
 			(effects
 				(font
@@
 		)
 		(property "Footprint" "Diode_SMD:D_SMA"
-			(at 97.79 20.955 0)
+			(at 54.61 17.145 0)
 			(effects
 				(font
@@
 		)
 		(property "Datasheet" "https://www.vishay.com/docs/88746/ss12.pdf"
-			(at 97.79 25.4 0)
+			(at 54.61 21.59 0)
 			(effects
 				(font
@@
 		)
 		(property "Description" "40V 1A Schottky Diode, SMA"
-			(at 97.79 25.4 0)
+			(at 54.61 21.59 0)
 			(effects
 				(font
@@
 	(symbol
 		(lib_id "power:+5V")
-		(at 104.14 24.13 0)
+		(at 99.06 24.13 0)
 		(unit 1)
 		(exclude_from_sim no)
@@
 		(fields_autoplaced yes)
 		(property "Reference" "#PWR013"
-			(at 104.14 27.94 0)
+			(at 99.06 27.94 0)
 			(effects
 				(font
@@
 		)
 		(property "Value" "+5V"
-			(at 104.14 19.05 0)
+			(at 99.06 19.05 0)
 			(effects
 				(font
@@
 		)
 		(property "Footprint" ""
-			(at 104.14 24.13 0)
+			(at 99.06 24.13 0)
 			(effects
 				(font
@@
 		)
 		(property "Datasheet" ""
-			(at 104.14 24.13 0)
+			(at 99.06 24.13 0)
 			(effects
 				(font
@@
 		)
 		(property "Description" "Power symbol creates a global label with name \"+5V\""
-			(at 104.14 24.13 0)
+			(at 99.06 24.13 0)
 			(effects
 				(font
@@
 	(symbol
 		(lib_id "Device:R_Small_US")
-		(at 40.64 31.75 0)
+		(at 44.45 33.02 0)
 		(unit 1)
 		(exclude_from_sim no)
@@
 		(dnp no)
 		(property "Reference" "R3"
-			(at 41.402 29.464 0)
+			(at 45.212 30.734 0)
 			(effects
 				(font
@@
 		)
 		(property "Value" "100k"
-			(at 41.402 33.782 0)
+			(at 45.212 35.052 0)
 			(effects
 				(font
@@
 		)
 		(property "Footprint" "Resistor_SMD:R_0603_1608Metric_Pad0.98x0.95mm_HandSolder"
-			(at 40.64 31.75 0)
+			(at 44.45 33.02 0)
 			(effects
 				(font
@@
 		)
 		(property "Datasheet" "~"
-			(at 40.64 31.75 0)
+			(at 44.45 33.02 0)
 			(effects
 				(font
@@
 		)
 		(property "Description" "Resistor, small US symbol"
-			(at 40.64 31.75 0)
+			(at 44.45 33.02 0)
 			(effects
 				(font

Commit message: change ldo to hand-solderable type
Parts:
- removed U2: TLV75733PDRV, Package_SON:WSON-6-1EP_2x2mm_P0.65mm_EP1x1.6mm, symbol Regulator_Linear:TLV75733PDRV
- added U2: TLV75733PDBV, Package_TO_SOT_SMD:SOT-23-5, symbol Regulator_Linear:TLV75733PDBV
Connections:
- net +3.3V: now also U2.5 (OUT)
- net +5V: now also U2.1 (IN)
- net GND: now also U2.2 (GND)
- net at R6.1: now also U2.3 (EN)
Changed lines of the file:
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@@
 	)
 	(symbol
-		(lib_id "Regulator_Linear:TLV75733PDRV")
-		(at 158.75 29.21 0)
-		(unit 1)
-		(exclude_from_sim no)
-		(in_bom yes)
-		(on_board yes)
-		(dnp no)
-		(fields_autoplaced yes)
-		(property "Reference" "U2"
-			(at 158.75 20.32 0)
-			(effects
-				(font
-					(size 1.27 1.27)
-				)
-			)
-		)
-		(property "Value" "TLV75733PDRV"
-			(at 158.75 22.86 0)
-			(effects
-				(font
-					(size 1.27 1.27)
-				)
-			)
-		)
-		(property "Footprint" "Package_SON:WSON-6-1EP_2x2mm_P0.65mm_EP1x1.6mm"
-			(at 158.75 20.955 0)
-			(effects
-				(font
-					(size 1.27 1.27)
-					(italic yes)
-				)
-				(hide yes)
-			)
-		)
-		(property "Datasheet" "https://www.ti.com/lit/ds/symlink/tlv757p.pdf"
-			(at 158.75 27.94 0)
-			(effects
-				(font
-					(size 1.27 1.27)
-				)
-				(hide yes)
-			)
-		)
-		(property "Description" "1A Low IQ Small Size Low Dropout Voltage Regulator, Fixed Output 3.3V, WSON6"
-			(at 158.75 29.21 0)
-			(effects
-				(font
-					(size 1.27 1.27)
-				)
-				(hide yes)
-			)
-		)
-		(pin "7"
-		)
-		(pin "4"
-		)
-		(pin "6"
-		)
-		(pin "5"
-		)
-		(pin "1"
-		)
-		(pin "3"
-		)
-		(pin "2"
-		)
-		(instances
-			(project "customDevboard"
-				(path "/87078d80-bd64-4f8e-8d0b-a79df4010aa3"
-					(reference "U2")
-					(unit 1)
-				)
-			)
-		)
-	)
-	(symbol
 		(lib_id "power:GND")
 		(at 44.45 38.1 0)
@@
 					(unit 1)
 				)
+			)
+		)
+	)
+	(symbol
+		(lib_id "Regulator_Linear:TLV75733PDBV")
+		(at 158.75 29.21 0)
+		(unit 1)
+		(exclude_from_sim no)
+		(in_bom yes)
+		(on_board yes)
+		(dnp no)
+		(fields_autoplaced yes)
+		(property "Reference" "U2"
+			(at 158.75 20.32 0)
+			(effects
+				(font
+					(size 1.27 1.27)
+				)
+			)
+		)
+		(property "Value" "TLV75733PDBV"
+			(at 158.75 22.86 0)
+			(effects
+				(font
+					(size 1.27 1.27)
+				)
+			)
+		)
+		(property "Footprint" "Package_TO_SOT_SMD:SOT-23-5"
+			(at 158.75 20.955 0)
+			(effects
+				(font
+					(size 1.27 1.27)
+					(italic yes)
+				)
+				(hide yes)
+			)
+		)
+		(property "Datasheet" "https://www.ti.com/lit/ds/symlink/tlv757p.pdf"
+			(at 158.75 27.94 0)
+			(effects
+				(font
+					(size 1.27 1.27)
+				)
+				(hide yes)
+			)
+		)
+		(property "Description" "1A Low IQ Small Size Low Dropout Voltage Regulator, Fixed Output 3.3V, SOT-23-5"
+			(at 158.75 29.21 0)
+			(effects
+				(font
+					(size 1.27 1.27)
+				)
+				(hide yes)
+			)
+		)
+		(pin "4"
+		)
+		(pin "2"
+		)
+		(pin "3"
+		)
+		(pin "5"
+		)
+		(pin "1"
+		)
+		(instances
+			(project ""
+				(path "/87078d80-bd64-4f8e-8d0b-a79df4010aa3"
+					(reference "U2")
+					(unit 1)
+				)
